File: Vaughn_Com/ComBoard/ComBoard.kicad_sch (KiCad schematic)
At the start: 9 parts, among them J1 Conn_01x06_Pin, Q1 2N3904, Q2 2N3904, U1 PIC16LF1938-I/SP

Commit message: this board is krzy
Parts:
- added D8: LED_Dual_AAK, symbol Device:LED_Dual_AAK
- added JP2, JP3: Screw_Terminal_01x04, symbol Connector:Screw_Terminal_01x04
- added RP1: 1M, Resistor_THT:R_Array_SIP6, symbol Device:R_Network05
- added RP2: 1k, Resistor_THT:R_Array_SIP8, symbol Device:R_Network07
Connections:
- net GND: now also U1.19 (VSS), U1.8 (VSS)
- net VCC: now also C1.1, J1.1 (Pin_1), U1.1 (VPP/*MCLR/RE3), U1.20 (VDD), JP2.2 (Pin_2), JP3.2 (Pin_2); no longer R1.1
- net TXA: now reaches Q1.3 (C)
- net TXA: now also JP2.3 (Pin_3)
- net mcu28: now reaches J1.4 (Pin_4)
- net mcu28: now also U1.28 (RB7/ICSPDAT/ICDDAT)
- net mcu27: now reaches J1.5 (Pin_5)
- net mcu27: now also U1.27 (RB6/ICSPCLK/ICDCLK)
- net mcu24: now reaches J1.6 (Pin_6)
- net mcu24: now also U1.24 (RB3)
- net TXB: now reaches Q2.3 (C)
- net TXB: now also JP3.3 (Pin_3)
- net mcu17: now reaches U1.17 (RC6)
- net mcu17: now also RP1.1 (common)
- new net: R1.1, R1.2
- new net RXA: JP2.4 (Pin_4)
- new net RXB: JP3.4 (Pin_4)
- new net led: D8.3 (K), RP1.6 (R5)
- new net mcu14: D8.1 (A1)
Other:
- note added: "0V"
- moved on the sheet: C1, Q1, Q2, R1, R2, U1
