File: Vaughn_HPC/Vaughn_HPC.kicad_sch (KiCad schematic)
At the start: 63 parts, among them J1 Conn_01x06_Pin, J10 1287, J11 1287, J12 1287, J12 1825640000, J13 1287, J13 1825640000, J14 1287, J14 1825640000, J15 1287, J15 1825640000, J16 1287, J16 1825640000, J17 1287, J2 AZ943-1CH-24DE, J3 AZ943-1CH-24DE, J4 AZ943-1CH-24DE, J5 1287, J6 1267, J7 1267, J8 1287, J9 1287, K1 AZ2100-1A-12DEF, Q1 2N3904, Q2 2N3904, Q3 2N3904, Q4 2N3904, Q5 BF244A, Q6 BF244A, Q7 BF244A, Q8 BF244A, U1 LM7805_TO220, U2 LM7812_TO220, U3 PIC16LF1938-I/SP

Commit message: shuffle
Parts:
- removed R8: 1K, symbol Device:R
Connections:
- net 5v: now also J1.5 (Pin_5), R7.1
Other:
- moved on the sheet: D8, J12, J13, J15, R9
Changed lines of the file:
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@@
 	(wire
 		(pts
-			(xy 217.17 186.69) (xy 184.15 186.69)
+			(xy 217.17 186.69) (xy 185.42 186.69)
 		)
 		(stroke
@@
 	(wire
 		(pts
-			(xy 363.22 138.43) (xy 351.79 138.43)
+			(xy 373.38 135.89) (xy 351.79 135.89)
 		)
 		(stroke
@@
 	(wire
 		(pts
+			(xy 185.42 212.09) (xy 186.69 212.09)
+		)
+		(stroke
+			(width 0)
+			(type default)
+		)
+	)
+	(wire
+		(pts
 			(xy 373.38 29.21) (xy 373.38 35.56)
 		)
@@
 	(wire
 		(pts
-			(xy 351.79 138.43) (xy 351.79 123.19)
+			(xy 351.79 135.89) (xy 351.79 123.19)
 		)
 		(stroke
@@
 	(wire
 		(pts
-			(xy 208.28 229.87) (xy 208.28 191.77)
+			(xy 208.28 214.63) (xy 208.28 191.77)
 		)
 		(stroke
@@
 	(wire
 		(pts
-			(xy 351.79 123.19) (xy 360.68 123.19)
-		)
-		(stroke
-			(width 0)
-			(type default)
-		)
-	)
-	(wire
-		(pts
 			(xy 173.99 312.42) (xy 193.04 312.42)
 		)
@@
 	(wire
 		(pts
-			(xy 62.23 176.53) (xy 62.23 189.23)
+			(xy 185.42 200.66) (xy 185.42 212.09)
 		)
 		(stroke
@@
 	(wire
 		(pts
-			(xy 144.78 66.04) (xy 144.78 72.39)
+			(xy 62.23 176.53) (xy 62.23 189.23)
 		)
 		(stroke
@@
 	(wire
 		(pts
-			(xy 308.61 161.29) (xy 316.23 161.29)
+			(xy 144.78 66.04) (xy 144.78 72.39)
 		)
 		(stroke
@@
 	(wire
 		(pts
-			(xy 200.66 274.32) (xy 218.44 274.32)
+			(xy 308.61 161.29) (xy 316.23 161.29)
 		)
 		(stroke
@@
 	(wire
 		(pts
-			(xy 184.15 227.33) (xy 186.69 227.33)
+			(xy 200.66 274.32) (xy 218.44 274.32)
 		)
 		(stroke
@@
 	(wire
 		(pts
-			(xy 201.93 229.87) (xy 208.28 229.87)
+			(xy 201.93 214.63) (xy 208.28 214.63)
 		)
 		(stroke
@@
 	(wire
 		(pts
-			(xy 355.6 86.36) (xy 351.79 86.36)
+			(xy 373.38 86.36) (xy 351.79 86.36)
 		)
 		(stroke
@@
 	(wire
 		(pts
-			(xy 184.15 186.69) (xy 184.15 204.47)
+			(xy 185.42 186.69) (xy 185.42 193.04)
 		)
 		(stroke
@@
 	(wire
 		(pts
-			(xy 205.74 224.79) (xy 205.74 189.23)
+			(xy 205.74 209.55) (xy 205.74 189.23)
+		)
+		(stroke
+			(width 0)
+			(type default)
+		)
+	)
+	(wire
+		(pts
+			(xy 351.79 123.19) (xy 373.38 123.19)
 		)
 		(stroke
@@
 	(wire
 		(pts
-			(xy 201.93 224.79) (xy 205.74 224.79)
+			(xy 201.93 209.55) (xy 205.74 209.55)
 		)
 		(stroke
@@
 	(wire
 		(pts
-			(xy 184.15 212.09) (xy 184.15 227.33)
-		)
-		(stroke
-			(width 0)
-			(type default)
-		)
-	)
-	(wire
-		(pts
 			(xy 308.61 186.69) (xy 311.15 186.69)
 		)
@@
 		)
 	)
+	(label "5v"
+		(at 317.5 45.72 0)
+		(effects
+			(font
+				(size 1.27 1.27)
+			)
+			(justify left bottom)
+		)
+	)
 	(label "mcu11_j16"
 		(at 360.68 35.56 0)
@@
 	(symbol
 		(lib_id "Device:LED_Dual_AAK")
-		(at 194.31 227.33 0)
+		(at 194.31 212.09 0)
 		(unit 1)
 		(exclude_from_sim no)
@@
 		(fields_autoplaced yes)
 		(property "Reference" "D8"
-			(at 194.3735 215.9 0)
+			(at 194.3735 200.66 0)
 			(effects
 				(font
@@
 		)
 		(property "Value" "LED_Dual_AAK"
-			(at 194.3735 218.44 0)
+			(at 194.3735 203.2 0)
 			(effects
 				(font
@@
 		)
 		(property "Footprint" ""
-			(at 194.31 227.33 0)
+			(at 194.31 212.09 0)
 			(effects
 				(font
@@
 		)
 		(property "Datasheet" "~"
-			(at 194.31 227.33 0)
+			(at 194.31 212.09 0)
 			(effects
 				(font
@@
 		)
 		(property "Description" "Dual LED, common cathode on pin 3"
-			(at 194.31 227.33 0)
+			(at 194.31 212.09 0)
 			(effects
 				(font
@@
 	(symbol
 		(lib_id "quickConnect:1825640000")
-		(at 355.6 78.74 0)
+		(at 373.38 78.74 0)
 		(unit 1)
 		(exclude_from_sim no)
@@
 		(fields_autoplaced yes)
 		(property "Reference" "J15"
-			(at 369.57 81.2799 0)
+			(at 387.35 81.2799 0)
 			(effects
 				(font
@@
 		)
 		(property "Value" "1825640000"
-			(at 369.57 83.8199 0)
+			(at 387.35 83.8199 0)
 			(effects
 				(font
@@
 		)
 		(property "Footprint" "CONN4_1825640000_WED"
-			(at 355.6 78.74 0)
+			(at 373.38 78.74 0)
 			(effects
 				(font
@@
 		)
 		(property "Datasheet" "1825640000"
-			(at 355.6 78.74 0)
+			(at 373.38 78.74 0)
 			(effects
 				(font
@@
 		)
 		(property "Description" ""
-			(at 355.6 78.74 0)
+			(at 373.38 78.74 0)
 			(effects
 				(font
@@
 	(symbol
 		(lib_id "quickConnect:1825640000")
-		(at 360.68 115.57 0)
+		(at 373.38 115.57 0)
 		(unit 1)
 		(exclude_from_sim no)
@@
 		(fields_autoplaced yes)
 		(property "Reference" "J13"
-			(at 374.65 118.1099 0)
+			(at 387.35 118.1099 0)
 			(effects
 				(font
@@
 		)
 		(property "Value" "1825640000"
-			(at 374.65 120.6499 0)
+			(at 387.35 120.6499 0)
 			(effects
 				(font
@@
 		)
 		(property "Footprint" "CONN4_1825640000_WED"
-			(at 360.68 115.57 0)
+			(at 373.38 115.57 0)
 			(effects
 				(font
@@
 		)
 		(property "Datasheet" "1825640000"
-			(at 360.68 115.57 0)
+			(at 373.38 115.57 0)
 			(effects
 				(font
@@
 		)
 		(property "Description" ""
-			(at 360.68 115.57 0)
+			(at 373.38 115.57 0)
 			(effects
 				(font
@@
 	(symbol
 		(lib_id "Device:R")
-		(at 184.15 208.28 0)
+		(at 185.42 196.85 0)
 		(unit 1)
 		(exclude_from_sim no)
@@
 		(fields_autoplaced yes)
 		(property "Reference" "R9"
-			(at 186.69 207.0099 0)
+			(at 187.96 195.5799 0)
 			(effects
 				(font
@@
 		)
 		(property "Value" "120"
-			(at 186.69 209.5499 0)
+			(at 187.96 198.1199 0)
 			(effects
 				(font
@@
 		)
 		(property "Footprint" ""
-			(at 182.372 208.28 90)
+			(at 183.642 196.85 90)
 			(effects
 				(font
@@
 		)
 		(property "Datasheet" "~"
-			(at 184.15 208.28 0)
+			(at 185.42 196.85 0)
 			(effects
 				(font
@@
 		)
 		(property "Description" "Resistor"
-			(at 184.15 208.28 0)
+			(at 185.42 196.85 0)
 			(effects
 				(font
@@
 	(symbol
 		(lib_id "quickConnect:1825640000")
-		(at 363.22 138.43 0)
+		(at 373.38 135.89 0)
 		(unit 1)
 		(exclude_from_sim no)
@@
 		(fields_autoplaced yes)
 		(property "Reference" "J12"
-			(at 377.19 140.9699 0)
+			(at 387.35 138.4299 0)
 			(effects
 				(font
@@
 		)
 		(property "Value" "1825640000"
-			(at 377.19 143.5099 0)
+			(at 387.35 140.9699 0)
 			(effects
 				(font
@@
 		)
 		(property "Footprint" "CONN4_1825640000_WED"
-			(at 363.22 138.43 0)
+			(at 373.38 135.89 0)
 			(effects
 				(font
@@
 		)
 		(property "Datasheet" "1825640000"
-			(at 363.22 138.43 0)
+			(at 373.38 135.89 0)
 			(effects
 				(font
@@
 		)
 		(property "Description" ""
-			(at 363.22 138.43 0)
+			(at 373.38 135.89 0)
 			(effects
 				(font
@@
 					(unit 1)
 				)
-			)
-		)
-	)
-	(symbol
-		(lib_id "Device:R")
-		(at 284.48 128.27 0)
-		(unit 1)
-		(exclude_from_sim no)
-		(in_bom yes)
-		(on_board yes)
-		(dnp no)
-		(fields_autoplaced yes)
-		(property "Reference" "R8"
-			(at 287.02 126.9999 0)
-			(effects
-				(font
-					(size 1.27 1.27)
-				)
-				(justify left)
-			)
-		)
-		(property "Value" "1K"
-			(at 287.02 129.5399 0)
-			(effects
-				(font
-					(size 1.27 1.27)
-				)
-				(justify left)
-			)
-		)
-		(property "Footprint" ""
-			(at 282.702 128.27 90)
-			(effects
-				(font
-					(size 1.27 1.27)
-				)
-				(hide yes)
-			)
-		)
-		(property "Datasheet" "~"
-			(at 284.48 128.27 0)
-			(effects
-				(font
-					(size 1.27 1.27)
-				)
-				(hide yes)
-			)
-		)
-		(property "Description" "Resistor"
-			(at 284.48 128.27 0)
-			(effects
-				(font
-					(size 1.27 1.27)
-				)
-				(hide yes)
-			)
-		)
-		(pin "2"
-		)
-		(pin "1"
-		)
-		(instances
-			(project ""
-				(path "/93c2951a-8c49-47b9-a2da-5f3676181e30"
-					(reference "R8")
-					(unit 1)
-				)

Commit message: preping for ERC check
1 Error.
Error input Power Pin Not driven by an Output Power Pin
Parts:
- removed J10, J13, J14, J5: 1287, 1287:KEYSTONE_1287, symbol spade2:1287
- removed RP1, RP2: R_Network08, Resistor_THT:R_Array_SIP9, symbol Device:R_Network08
- added RP1, RP2: R_Network07, Resistor_THT:R_Array_SIP8, symbol Device:R_Network07
- renumbered J16 to J1, J17 to J2, J8 to J3, J9 to J4, J11 to J5, J12 to J6, J15 to J7, J6 to J8, J7 to J9, J1 to JP3, K1 to RLY1, J2 to RLY2, J3 to RLY3, J4 to RLY4
Connections:
- net 12v is gone; now on net 12V: JP4.1 (Pin_1)
- net prog1_j14 is gone; now on net mcu24: J14.1, JP3.1 (Pin_1)
- net 5V: now also C4.1, JP3.5 (Pin_5), R7.1, U3.20 (VDD)
- net 5v: now also RP2.4 (R3), RP2.5 (R4), RP2.8 (R7); no longer C4.1, JP3.5 (Pin_5), R7.1, U3.20 (VDD)
- net RP1_2_Q2_base: now also RP1.2 (R1)
- net RP1_3_mcu15: now also RP1.3 (R2)
- net RP1_4_q3_base: now also RP1.4 (R3)
- net RP1_5_mcu16: now also RP1.5 (R4)
- net RP1_6_q4_base: now also RP1.6 (R5)
- net RP1_7_mcu10: now also RP1.7 (R6)
- net RP1_8_q1_base: now also Q1.2 (B), RP1.8 (R7)
- net RP2_3_q1_Emitter: now also RP2.2 (R1), RP2.3 (R2)
- net mcu9_array1: now also RP1.1 (common)
- net prog6_mcu1: now also RP2.6 (R5)
- net mcu2: now reaches R3.1, U3.2 (RA0)
- net mcu2: now also J12.4
- net mcu5: now reaches J15.1
- net mcu5: now also R2.1, U3.5 (RA3)
- net mcu3: now reaches R4.2, U3.3 (RA1)
- net mcu3: now also J13.1
- net J6: now reaches RLY4.1 (COM)
- net J6: now also J6.1_2
- net mcu24: now reaches R5.1, U3.24 (RB3)
- net jp2_3: now reaches JP2.3 (Pin_3), R11.2
- net jp2_3: now also RP2.7 (R6)
- net RP1_1_mcu6 renamed RP2_1_mcu6
- net RP2_1_mcu6: now also RP2.1 (common)
- no-connect marks 0 -> 19
Other:
- moved on the sheet: Q2, Q3, Q4, R11

Commit message: updates
Connections:
- net at RV1.1, TR1.1: now also J1.1_2; no longer J1.1_1
- net at RV1.2, TR1.4: now also J2.1_1; no longer J2.1_2
Other:
- moved on the sheet: C1, C2, C3, C4, D1, D2, D3, D4, D5, D6, D7, D8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
